File: Hardware/R3_0/BlastGateRev3_1/BlastGateRev3_1/BlastGateRev3_1.kicad_pcb (KiCad board)
At the start: 2 copper layers, 50.8 x 44.5 mm, 44 parts, among them J1 Conn_01x03_Male, J2 Conn_01x06_Male, J3 USB_B_Micro, J4 RJ9, J5 Conn_01x03_Male, SW1 SW_DIP_x03, SW2 SW_SPDT_MSM, SW4 SW_SPDT_MSM, U1 AP2112M-3.3, U2 ESP32-WROOM-32D

Commit message: Add GC, Code Cleanup
Parts:
- moved D6 10.9 mm to (117.5, 157.5)
- moved PROG1 9.28 mm to (105.0, 157.9)
Routing:
- net /RXD: track 7.33 -> 20.7 mm
- net GND: track 50.1 -> 61.6 mm
- net /GPIO_0: track 3.95 -> 10.9 mm
- net /RXD_5V: track 6.07 -> 12.6 mm
- net /MODE: track 48.4 -> 47.3 mm
- net /MAN_ON: track 30.0 -> 31.2 mm
